Commit message: Update 01-myfirst.urdf

File: tutorial_ws/urdf/01-myfirst.urdf (robot description, URDF)
Before this commit: robot visual, 16 links, 15 joints
Links:
- removed link box
- removed link gripper_pole
- removed link head
- removed link left_base
- removed link left_gripper
- removed link left_leg
- removed link left_tip
- removed link right_base
- removed link right_gripper
- removed link right_leg
- removed link right_tip
Joints:
- removed joint base_to_left_leg
- removed joint base_to_right_leg
- removed joint gripper_extension
- removed joint head_swivel
- removed joint left_base_joint
- removed joint left_gripper_joint
- removed joint left_tip_joint
- removed joint right_base_joint
- removed joint right_gripper_joint
- removed joint right_tip_joint
- removed joint tobox
- joint left_back_wheel_joint: axis (none) -> 1 0 1; origin xyz=-0.133333333333 0 -0.085 rpy=0 0 0 -> xyz=-0.133333333333 -0.2 -0.085; parent left_base -> base_link; type fixed -> continuous
- joint left_front_wheel_joint: axis (none) -> 1 0 1; origin xyz=0.133333333333 0 -0.085 rpy=0 0 0 -> xyz=0.133333333333 -0.2 -0.085; parent left_base -> base_link; type fixed -> continuous
- joint right_back_wheel_joint: axis (none) -> 1 0 1; origin xyz=-0.133333333333 0 -0.085 rpy=0 0 0 -> xyz=-0.133333333333 0.2 -0.085; parent right_base -> base_link; type fixed -> continuous
- joint right_front_wheel_joint: axis (none) -> 1 0 1; origin xyz=0.133333333333 0 -0.085 rpy=0 0 0 -> xyz=0.133333333333 0.2 -0.085; parent right_base -> base_link; type fixed -> continuous
